File: USB2TTL-CH340G.sch (KiCad schematic (older format))
At the start: 20 parts, among them P1 USB_OTG, P2 PWR_SEL, P3 CONN_01X06, U1 CH340G, X1 CRYSTAL_SMD

Commit message: 1.新建myRegul库并添加元件LDO芯片XP6206；2.用最大可提供500mA电流的XP6206替换掉原来的二极管稳压电路，提高稳定性；3.调整PCB元件布局。
Parts:
- removed C4: 10uF, Capacitors_SMD:C_0603, symbol CP
- removed D4: 3V3, Diodes_SMD:SOD-123, symbol D
- removed R3: 200, Resistors_SMD:R_0603, symbol R
- added C3, C5: 1uF, Capacitors_SMD:C_0603, symbol C
- added U1: XC6206P332MR, TO_SOT_Packages_SMD:SOT-23, symbol XC6206P332MR
- renumbered C3 to C4, C5 to C6, C6 to C7, C7 to C8, R4 to R3, U1 to U2
Connections:
- wire segments 58 -> 59
Other:
- moved on the sheet: C1, C2
Changed lines of the file:
@@
 LIBS:valves
 LIBS:ch340g
+LIBS:myRegul
 LIBS:USB2TTL-CH340G-cache
 EELAYER 25 0
@@
 L CP C1
 U 1 1 57500D41
-P 3300 2850
-F 0 "C1" H 3325 2950 50  0000 L CNN
-F 1 "10uF" H 3325 2750 50  0000 L CNN
-F 2 "Capacitors_SMD:C_0603" H 3338 2700 50  0001 C CNN
-F 3 "" H 3300 2850 50  0000 C CNN
-	1    3300 2850
-	1    0    0    -1
-$EndComp
-$Comp
-L CP C4
-U 1 1 57500D89
-P 4750 2850
-F 0 "C4" H 4775 2950 50  0000 L CNN
-F 1 "10uF" H 4775 2750 50  0000 L CNN
-F 2 "Capacitors_SMD:C_0603" H 4788 2700 50  0001 C CNN
-F 3 "" H 4750 2850 50  0000 C CNN
-	1    4750 2850
+P 3100 2850
+F 0 "C1" H 3125 2950 50  0000 L CNN
+F 1 "10uF" H 3125 2750 50  0000 L CNN
+F 2 "Capacitors_SMD:C_0603" H 3138 2700 50  0001 C CNN
+F 3 "" H 3100 2850 50  0000 C CNN
+	1    3100 2850
 	1    0    0    -1
 $EndComp
@@
 L C C2
 U 1 1 57500DBB
-P 3700 2850
-F 0 "C2" H 3725 2950 50  0000 L CNN
-F 1 "0.1uF" H 3725 2750 50  0000 L CNN
-F 2 "Capacitors_SMD:C_0603" H 3738 2700 50  0001 C CNN
-F 3 "" H 3700 2850 50  0000 C CNN
-	1    3700 2850
-	1    0    0    -1
-$EndComp
-$Comp
-L R R3
-U 1 1 57500E03
-P 4050 2600
-F 0 "R3" V 4130 2600 50  0000 C CNN
-F 1 "200" V 4050 2600 50  0000 C CNN
-F 2 "Resistors_SMD:R_0603" V 3980 2600 50  0001 C CNN
-F 3 "" H 4050 2600 50  0000 C CNN
-	1    4050 2600
-	0    1    1    0
+P 3500 2850
+F 0 "C2" H 3525 2950 50  0000 L CNN
+F 1 "0.1uF" H 3525 2750 50  0000 L CNN
+F 2 "Capacitors_SMD:C_0603" H 3538 2700 50  0001 C CNN
+F 3 "" H 3500 2850 50  0000 C CNN
+	1    3500 2850
+	1    0    0    -1
 $EndComp
 $Comp
@@
 $EndComp
 $Comp
-L R R4
+L R R3
 U 1 1 57500F93
 P 4050 4500
-F 0 "R4" V 4130 4500 50  0000 C CNN
+F 0 "R3" V 4130 4500 50  0000 C CNN
 F 1 "4.7K" V 4050 4500 50  0000 C CNN
 F 2 "Resistors_SMD:R_0603" V 3980 4500 50  0001 C CNN
@@
 $EndComp
 $Comp
-L C C3
+L C C4
 U 1 1 57500FCD
 P 4400 4500
-F 0 "C3" H 4425 4600 50  0000 L CNN
+F 0 "C4" H 4425 4600 50  0000 L CNN
 F 1 "0.1uF" H 4425 4400 50  0000 L CNN
 F 2 "Capacitors_SMD:C_0603" H 4438 4350 50  0001 C CNN
@@
 $EndComp
 $Comp
-L GND #PWR1
+L GND #PWR01
 U 1 1 5750100D
 P 3350 5550
-F 0 "#PWR1" H 3350 5300 50  0001 C CNN
+F 0 "#PWR01" H 3350 5300 50  0001 C CNN
 F 1 "GND" H 3350 5400 50  0000 C CNN
 F 2 "" H 3350 5550 50  0000 C CNN
@@
 $EndComp
 $Comp
-L GND #PWR5
+L GND #PWR02
 U 1 1 5750103D
 P 4400 5050
-F 0 "#PWR5" H 4400 4800 50  0001 C CNN
+F 0 "#PWR02" H 4400 4800 50  0001 C CNN
 F 1 "GND" H 4400 4900 50  0000 C CNN
 F 2 "" H 4400 5050 50  0000 C CNN
@@
 $EndComp
 $Comp
-L GND #PWR8
+L GND #PWR03
 U 1 1 57501066
 P 6400 5700
-F 0 "#PWR8" H 6400 5450 50  0001 C CNN
+F 0 "#PWR03" H 6400 5450 50  0001 C CNN
 F 1 "GND" H 6400 5550 50  0000 C CNN
 F 2 "" H 6400 5700 50  0000 C CNN
@@
 $EndComp
 $Comp
-L GND #PWR9
+L GND #PWR04
 U 1 1 575010D5
 P 7150 5700
-F 0 "#PWR9" H 7150 5450 50  0001 C CNN
+F 0 "#PWR04" H 7150 5450 50  0001 C CNN
 F 1 "GND" H 7150 5550 50  0000 C CNN
 F 2 "" H 7150 5700 50  0000 C CNN
@@
 $EndComp
 $Comp
-L C C5
+L C C6
 U 1 1 57501211
 P 6400 5450
-F 0 "C5" H 6425 5550 50  0000 L CNN
+F 0 "C6" H 6425 5550 50  0000 L CNN
 F 1 "22pF" H 6425 5350 50  0000 L CNN
 F 2 "Capacitors_SMD:C_0603" H 6438 5300 50  0001 C CNN
@@
 $EndComp
 $Comp
-L C C7
+L C C8
 U 1 1 57501276
 P 7150 5450
-F 0 "C7" H 7175 5550 50  0000 L CNN
+F 0 "C8" H 7175 5550 50  0000 L CNN
 F 1 "22pF" H 7175 5350 50  0000 L CNN
 F 2 "Capacitors_SMD:C_0603" H 7188 5300 50  0001 C CNN
@@
 $EndComp
 $Comp
-L D D4
-U 1 1 575014DA
-P 4400 2850
-F 0 "D4" H 4400 2950 50  0000 C CNN
-F 1 "3V3" H 4400 2750 50  0000 C CNN
-F 2 "Diodes_SMD:SOD-123" H 4400 2850 50  0001 C CNN
-F 3 "" H 4400 2850 50  0000 C CNN
-	1    4400 2850
-	0    1    1    0
-$EndComp
-$Comp
-L GND #PWR4
+L GND #PWR05
 U 1 1 5750155B
-P 4400 3200
-F 0 "#PWR4" H 4400 2950 50  0001 C CNN
-F 1 "GND" H 4400 3050 50  0000 C CNN
-F 2 "" H 4400 3200 50  0000 C CNN
-F 3 "" H 4400 3200 50  0000 C CNN
-	1    4400 3200
-	1    0    0    -1
-$EndComp
-$Comp
-L VCC #PWR2
+P 4300 3200
+F 0 "#PWR05" H 4300 2950 50  0001 C CNN
+F 1 "GND" H 4300 3050 50  0000 C CNN
+F 2 "" H 4300 3200 50  0000 C CNN
+F 3 "" H 4300 3200 50  0000 C CNN
+	1    4300 3200
+	1    0    0    -1
+$EndComp
+$Comp
+L VCC #PWR06
 U 1 1 5750585A
 P 3700 4100
-F 0 "#PWR2" H 3700 3950 50  0001 C CNN
+F 0 "#PWR06" H 3700 3950 50  0001 C CNN
 F 1 "VCC" H 3700 4250 50  0000 C CNN
 F 2 "" H 3700 4100 50  0000 C CNN
@@
 $EndComp
 $Comp
-L VCC #PWR3
+L VCC #PWR07
 U 1 1 575058E8
 P 4050 4100
-F 0 "#PWR3" H 4050 3950 50  0001 C CNN
+F 0 "#PWR07" H 4050 3950 50  0001 C CNN
 F 1 "VCC" H 4050 4250 50  0000 C CNN
 F 2 "" H 4050 4100 50  0000 C CNN
@@
 RXD
 $Comp
-L VCC #PWR10
+L VCC #PWR08
 U 1 1 575060EC
 P 8450 4200
-F 0 "#PWR10" H 8450 4050 50  0001 C CNN
+F 0 "#PWR08" H 8450 4050 50  0001 C CNN
 F 1 "VCC" H 8450 4350 50  0000 C CNN
 F 2 "" H 8450 4200 50  0000 C CNN
@@
 DTR
 $Comp
-L CH340G U1
+L CH340G U2
 U 1 1 57504C18
 P 7800 4650
-F 0 "U1" H 7800 4150 60  0000 C CNN
+F 0 "U2" H 7800 4150 60  0000 C CNN
 F 1 "CH340G" H 7800 5150 60  0000 C CNN
 F 2 "SMD_Packages:SO-16-N" H 8000 4000 60  0001 C CNN
@@
 DTR
 $Comp
-L PWR_FLAG #FLG2
+L PWR_FLAG #FLG09
 U 1 1 57508993
 P 6300 2650
-F 0 "#FLG2" H 6300 2745 50  0001 C CNN
+F 0 "#FLG09" H 6300 2745 50  0001 C CNN
 F 1 "PWR_FLAG" H 6300 2830 50  0000 C CNN
 F 2 "" H 6300 2650 50  0000 C CNN
@@
 $EndComp
 $Comp
-L VCC #PWR7
+L VCC #PWR010
 U 1 1 57508B09
 P 6300 2900
-F 0 "#PWR7" H 6300 2750 50  0001 C CNN
+F 0 "#PWR010" H 6300 2750 50  0001 C CNN
 F 1 "VCC" H 6300 3050 50  0000 C CNN
 F 2 "" H 6300 2900 50  0000 C CNN
@@
 NoConn ~ 5600 4300
 $Comp
-L PWR_FLAG #FLG1
+L PWR_FLAG #FLG011
 U 1 1 5750AEC9
 P 5700 2650
-F 0 "#FLG1" H 5700 2745 50  0001 C CNN
+F 0 "#FLG011" H 5700 2745 50  0001 C CNN
 F 1 "PWR_FLAG" H 5700 2830 50  0000 C CNN
 F 2 "" H 5700 2650 50  0000 C CNN
@@
 $EndComp
 $Comp
-L GND #PWR6
+L GND #PWR012
 U 1 1 5750AF10
 P 5700 2900
-F 0 "#PWR6" H 5700 2650 50  0001 C CNN
+F 0 "#PWR012" H 5700 2650 50  0001 C CNN
 F 1 "GND" H 5700 2750 50  0000 C CNN
 F 2 "" H 5700 2900 50  0000 C CNN
@@
 NoConn ~ 6000 4600
 Wire Wire Line
-	3300 2500 3300 2700
-Wire Wire Line
-	3300 2600 3900 2600
-Connection ~ 3300 2600
-Wire Wire Line
-	4200 2600 4750 2600
+	3100 2500 3100 2700
+Wire Wire Line
+	3100 2600 3900 2600
+Connection ~ 3100 2600
 Wire Wire Line
 	4750 2500 4750 2700
 Connection ~ 4750 2600
-Wire Wire Line
-	4400 2700 4400 2600
-Connection ~ 4400 2600
-Wire Wire Line
-	3700 2700 3700 2600
-Connection ~ 3700 2600
-Wire Wire Line
-	3300 3000 3300 3100
-Wire Wire Line
-	3300 3100 4750 3100
-Wire Wire Line
-	4400 3000 4400 3200
-Connection ~ 4400 3100
-Wire Wire Line
-	3700 3000 3700 3100
-Connection ~ 3700 3100
+Connection ~ 3500 2600
+Wire Wire Line
+	3100 3000 3100 3100
+Wire Wire Line
+	3500 3000 3500 3100
+Connection ~ 3500 3100
 Wire Wire Line
 	4750 3100 4750 3000
@@
 Wire Wire Line
 	6000 4500 6500 4500
-Text GLabel 3300 2500 1    60   Input ~ 0
+Text GLabel 3100 2500 1    60   Input ~ 0
 +5V
 Wire Wire Line
@@
 	6950 4600 7300 4600
 $Comp
-L C C6
+L C C7
 U 1 1 575D2FE6
 P 6650 4500
-F 0 "C6" V 6550 4350 50  0000 L CNN
+F 0 "C7" V 6550 4350 50  0000 L CNN
 F 1 "0.01uF" V 6800 4400 50  0000 L CNN
 F 2 "Capacitors_SMD:C_0603" H 6688 4350 50  0001 C CNN
@@
 Text Label 8450 4300 2    60   ~ 0
 VCC
+Wire Wire Line
+	3100 3100 4750 3100
+Wire Wire Line
+	4300 3200 4300 2900
+Connection ~ 4300 3100
+$Comp
+L C C3
+U 1 1 57B94B00
+P 3850 2850
+F 0 "C3" H 3875 2950 50  0000 L CNN
+F 1 "1uF" H 3875 2750 50  0000 L CNN
+F 2 "Capacitors_SMD:C_0603" H 3888 2700 50  0001 C CNN
+F 3 "" H 3850 2850 50  0000 C CNN
+	1    3850 2850
+	1    0    0    -1
+$EndComp
+Wire Wire Line
+	3850 2700 3850 2600
+Connection ~ 3850 2600
+Wire Wire Line
+	3850 3000 3850 3100
+Connection ~ 3850 3100
+$Comp
+L C C5
+U 1 1 57B94D18
+P 4750 2850
+F 0 "C5" H 4775 2950 50  0000 L CNN
+F 1 "1uF" H 4775 2750 50  0000 L CNN
+F 2 "Capacitors_SMD:C_0603" H 4788 2700 50  0001 C CNN
+F 3 "" H 4750 2850 50  0000 C CNN
+	1    4750 2850
+	1    0    0    -1
+$EndComp
+Wire Wire Line
+	4700 2600 4750 2600
+Wire Wire Line
+	3500 2700 3500 2600
+$Comp
+L XC6206P332MR U1
+U 1 1 57B95926
+P 4300 2650
+F 0 "U1" H 4300 2950 50  0000 C CNN
+F 1 "XC6206P332MR" H 4300 2850 50  0000 C CNN
+F 2 "TO_SOT_Packages_SMD:SOT-23" H 4300 2750 50  0001 C CIN
+F 3 "" H 4300 2650 50  0000 C CNN
+	1    4300 2650
+	1    0    0    -1
+$EndComp
 $EndSCHEMATC
